Commit message: update new leap

File: src/curobo/content/assets/robot/leap_hand/dual_dummy_arm_leap.urdf (robot description, URDF)
Before this commit: robot dual_dummy_arm_leap, 76 links, 75 joints
Joints:
- joint lh_joint_12: child lh_thumb_pip -> lh_pip_4; limit lower=-2.094 upper=0.349 effort=0.95 velocity=8.48 -> lower=-2.443 upper=0.47 effort=0.95 velocity=8.48; origin xyz=-1.0148132334464321502e-16 -0.014100000000000126321 -0.012999999999999956035 rpy=-1.570796326794896336 -1.570796326794896336 0 -> xyz=-0.14487422493839263726 -0.090040011501137440231 0.004900888583899039308 rpy=3.5629789726327258012e-15 1.5707963267948961139 0; parent lh_pip_4 -> lh_palm_lower_left
- joint lh_joint_13: child lh_pip_4 -> lh_thumb_pip; limit lower=-2.443 upper=0.47 effort=0.95 velocity=8.48 -> lower=-2.094 upper=0.349 effort=0.95 velocity=8.48; origin xyz=-0.14487422493839263726 -0.090040011501137440231 0.004900888583899039308 rpy=3.5629789726327258012e-15 1.5707963267948961139 0 -> xyz=-1.0148132334464321502e-16 -0.014100000000000126321 -0.012999999999999956035 rpy=-1.570796326794896336 -1.570796326794896336 0; parent lh_palm_lower_left -> lh_pip_4
